Commit message: too much work

File: mobile-base/mobile_base_description/urdf/base/model.xacro (robot description, xacro)
@@ -6,12 +6,13 @@
   <link name="base_footprint" />
   <joint name="chassis_link_joint" type="fixed">
-    <origin xyz="0 0 0.05" rpy="0 0 0" />
+    <!-- <origin xyz="0 0 0.1" rpy="0 0 0" /> -->
     <parent link="base_footprint"/>
     <child link="chassis_link" />
   </joint>
+  <xacro:property name="chassis_z" value="0.35" />
   <!-- chassis link -->
   <link name="chassis_link">
     <visual>
-      <origin xyz="0 0 .3" rpy="0 0 0" />
+      <origin xyz="0 0 ${chassis_z}" rpy="0 0 0" />
       <geometry>
         <!-- <box size="${base_dimensions}"/> -->
@@ -20,5 +21,5 @@
     </visual>
     <collision>
-      <origin xyz="0 0 .3"/>
+      <origin xyz="0 0 ${chassis_z}"/>
       <geometry>
         <box size="${base_dimensions}"/>
@@ -37,8 +38,12 @@
   <!-- Attach wheels -->
   <xacro:include filename="$(find mobile_base_description)/urdf/wheel/wheel.xacro" />
-  <xacro:wheel_macro index="1" parent="chassis_link" origin=".4 .4 .08"/>
+  <!-- <xacro:wheel_macro index="1" parent="chassis_link" origin=".4 .4 .08"/>
   <xacro:wheel_macro index="2" parent="chassis_link" origin=".4 -.4 .08"/>
   <xacro:wheel_macro index="3" parent="chassis_link" origin="-.4 -.4 .08"/>
-  <xacro:wheel_macro index="4" parent="chassis_link" origin="-.4 .4 .08"/>
+  <xacro:wheel_macro index="4" parent="chassis_link" origin="-.4 .4 .08"/> -->
+  <xacro:wheel_macro index="1" parent="chassis_link" origin=".179898 .28424 ${chassis_z - 0.208}"/>
+  <xacro:wheel_macro index="2" parent="chassis_link" origin=".179898 -.28424 ${chassis_z - 0.208}"/>
+  <xacro:wheel_macro index="3" parent="chassis_link" origin="-.5436278 .28424 ${chassis_z - 0.208}"/>
+  <xacro:wheel_macro index="4" parent="chassis_link" origin="-.5436278 -.28424 ${chassis_z - 0.208}"/>
   <!-- Load gazebo file-->
   <xacro:include filename="$(find mobile_base_description)/urdf/base/model.gazebo" />

File: mobile-base/mobile_base_description/urdf/wheel/wheel.xacro (robot description, xacro)
@@ -8,15 +8,17 @@
       <parent link="${parent}"/>
       <child link="wheel_${index}" />
-      <axis xyz="0 1 0"/>
+      <axis xyz="1 0 0"/>
     </joint>
     <link name="wheel_${index}">
       <visual>
-        <origin xyz=".0795 -.078 -.113" rpy="0 0 ${PI/2}" />
+        <!-- <origin xyz=".0795 -.078 -.113" rpy="0 0 ${PI/2}" /> -->
+        <origin xyz="0 0 0" rpy="0 0 ${PI/2}" />
         <geometry>
-          <mesh filename="$(find mobile_base_description)/meshes/mecanum_wheel.STL" scale="0.001 0.001 0.001"/>
+          <mesh filename="$(find mobile_base_description)/meshes/WPI_Mecanum_Wheel_fixed_origin.stl" scale="0.001 0.001 0.001"/>
         </geometry>
       </visual>
+          <!-- <origin xyz="0 0 0" rpy="${PI/2} 0 0"/> might have to rotate if wheel is flipped -->
       <collision>
-        <origin xyz="0 0 0" rpy="${PI/2} 0 0"/> <!--might have to rotate if wheel is flipped-->
+        <origin xyz="0 0 0" rpy="0 0 ${PI/2}"/>
         <geometry>
           <cylinder radius="${wheel_radius}" length="${wheel_width}"/>
@@ -34,11 +36,24 @@
     </link>
     <!-- <transmission name="wheel_${index}_joint_transmission">
+      <type>transmission_interface/SimpleTransmission</type>
+      <joint name="wheel_${index}_joint">
+          <hardwareInterface>hardware_interface/EffortJointInterface</hardwareInterface>
+      </joint>
+      <actuator name="wheel_${index}_joint_motor"> -->
+          <!-- <hardwareInterface>hardware_interface/EffortJointInterface</hardwareInterface> -->
+          <!-- <mechanicalReduction>1</mechanicalReduction>
+      </actuator>
+    </transmission> -->
+      <!-- Load Mecanum Wheel Motors -->
+  <!-- <xacro:macro name="wheel_motor_xacro" params="motor " />
+  <transmission name="motor_1_trans">
     <type>transmission_interface/SimpleTransmission</type>
-    <joint name="wheel_${index}_joint">
+    <joint name="wheel_1_joint">
         <hardwareInterface>hardware_interface/EffortJointInterface</hardwareInterface>
     </joint>
-    <actuator name="wheel_${index}_joint_motor">
+    <actuator name="wheel_1_joint_motor">
         <mechanicalReduction>1</mechanicalReduction>
-    </actuator> -->
+    </actuator>
+  </transmission> -->
     <gazebo reference="wheel_${index}">
       <mu1 value="0.0"/>

File: mobile-base/panda_arm/franka_description/robots/panda_arm.xacro (robot description, xacro)
@@ -209,8 +209,8 @@
       <type>transmission_interface/SimpleTransmission</type>
       <joint name="${arm_id}_joint1">
-	<hardwareInterface>hardware_interface/EffortJointInterface</hardwareInterface>
+	<hardwareInterface>hardware_interface/VelocityJointInterface</hardwareInterface>
       </joint>
       <actuator name="motor1">
-	<hardwareInterface>hardware_interface/EffortJointInterface</hardwareInterface>
+	<hardwareInterface>hardware_interface/VelocityJointInterface</hardwareInterface>
 	<mechanicalReduction>1</mechanicalReduction>
       </actuator>
@@ -219,8 +219,8 @@
       <type>transmission_interface/SimpleTransmission</type>
       <joint name="${arm_id}_joint2">
-	<hardwareInterface>hardware_interface/EffortJointInterface</hardwareInterface>
+	<hardwareInterface>hardware_interface/VelocityJointInterface</hardwareInterface>
       </joint>
       <actuator name="motor2">
-	<hardwareInterface>hardware_interface/EffortJointInterface</hardwareInterface>
+	<hardwareInterface>hardware_interface/VelocityJointInterface</hardwareInterface>
 	<mechanicalReduction>1</mechanicalReduction>
       </actuator>
@@ -229,8 +229,8 @@
       <type>transmission_interface/SimpleTransmission</type>
       <joint name="${arm_id}_joint3">
-	<hardwareInterface>hardware_interface/EffortJointInterface</hardwareInterface>
+	<hardwareInterface>hardware_interface/VelocityJointInterface</hardwareInterface>
       </joint>
       <actuator name="motor3">
-	<hardwareInterface>hardware_interface/EffortJointInterface</hardwareInterface>
+	<hardwareInterface>hardware_interface/VelocityJointInterface</hardwareInterface>
 	<mechanicalReduction>1</mechanicalReduction>
       </actuator>
@@ -239,8 +239,8 @@
       <type>transmission_interface/SimpleTransmission</type>
       <joint name="${arm_id}_joint4">
-	<hardwareInterface>hardware_interface/EffortJointInterface</hardwareInterface>
+	<hardwareInterface>hardware_interface/VelocityJointInterface</hardwareInterface>
       </joint>
       <actuator name="motor4">
-	<hardwareInterface>hardware_interface/EffortJointInterface</hardwareInterface>
+	<hardwareInterface>hardware_interface/VelocityJointInterface</hardwareInterface>
 	<mechanicalReduction>1</mechanicalReduction>
       </actuator>
@@ -249,8 +249,8 @@
       <type>transmission_interface/SimpleTransmission</type>
       <joint name="${arm_id}_joint5">
-	<hardwareInterface>hardware_interface/EffortJointInterface</hardwareInterface>
+	<hardwareInterface>hardware_interface/VelocityJointInterface</hardwareInterface>
       </joint>
       <actuator name="motor5">
-	<hardwareInterface>hardware_interface/EffortJointInterface</hardwareInterface>
+	<hardwareInterface>hardware_interface/VelocityJointInterface</hardwareInterface>
 	<mechanicalReduction>1</mechanicalReduction>
       </actuator>
@@ -259,8 +259,8 @@
       <type>transmission_interface/SimpleTransmission</type>
       <joint name="${arm_id}_joint6">
-	<hardwareInterface>hardware_interface/EffortJointInterface</hardwareInterface>
+	<hardwareInterface>hardware_interface/VelocityJointInterface</hardwareInterface>
       </joint>
       <actuator name="motor6">
-	<hardwareInterface>hardware_interface/EffortJointInterface</hardwareInterface>
+	<hardwareInterface>hardware_interface/VelocityJointInterface</hardwareInterface>
 	<mechanicalReduction>1</mechanicalReduction>
       </actuator>
@@ -269,8 +269,8 @@
       <type>transmission_interface/SimpleTransmission</type>
       <joint name="${arm_id}_joint7">
-	<hardwareInterface>hardware_interface/EffortJointInterface</hardwareInterface>
+	<hardwareInterface>hardware_interface/VelocityJointInterface</hardwareInterface>
       </joint>
       <actuator name="motor7">
-	<hardwareInterface>hardware_interface/EffortJointInterface</hardwareInterface>
+	<hardwareInterface>hardware_interface/VelocityJointInterface</hardwareInterface>
 	<mechanicalReduction>1</mechanicalReduction>
       </actuator>

File: mobile-base/panda_arm/panda_insert/panda_insert_description/urdf/panda_insert.xacro (robot description, xacro)
@@ -3,5 +3,13 @@
   <xacro:arg name="origin" default="0 0 1" />
   <xacro:include filename="$(find franka_description)/robots/panda_arm_hand.urdf.xacro" />
+  <!-- <xacro:include filename="$(find mobile_base_description)/urdf/base/model.xacro" /> -->
   <link name="world" />
+  <!-- <joint name="chassis_MI_joint" type="prismatic">
+    <origin xyz="0 0 -1"/>
+    <parent link="insert_link"/>
+    <child link="chassis_link" />
+    <axis xyz="0 0 1"/>
+    <limit effort="1000" lower="-1000" upper="1000" velocity="2" />
+  </joint> -->
   <joint name="insert_link_joint" type="fixed">
     <origin xyz="0 0 0" rpy="0 0 0" />

Commit message: Readjusted parallel linkage in Panda_description and Xacro files, adding in advanced position joint limits

File: mobile-base/mobile_base_description/urdf/base/model.xacro (robot description, xacro)
@@ -99,3 +99,9 @@
     </actuator>
   </transmission>
+  <!-- <gazebo>
+    <plugin name="gazebo_ros_control" filename="libgazebo_ros_control.so">
+      <robotNamespace>/base</robotNamespace>
+      <robotSimType>gazebo_ros_control/DefaultRobotHWSim</robotSimType>
+    </plugin>
+  </gazebo> -->
 </robot>

File: mobile-base/panda_arm/panda_insert/panda_insert_description/urdf/panda_insert.xacro (robot description, xacro)
@@ -1,19 +1,19 @@
 <?xml version="1.0"?>
 <robot name="panda_insert" xmlns:xacro="http://ros.org/wiki/xacro">
-  <xacro:arg name="origin" default="0 0 1" />
+  <xacro:arg name="origin" default="-0.05387925 0 1" />
   <xacro:include filename="$(find franka_description)/robots/panda_arm_hand.urdf.xacro" />
   <!-- <xacro:include filename="$(find mobile_base_description)/urdf/base/model.xacro" /> -->
   <link name="world" />
   <!-- <joint name="chassis_MI_joint" type="prismatic">
-    <origin xyz="0 0 -1"/>
+    <origin xyz="0 0 0.5" rpy="0 0 0"/>
     <parent link="insert_link"/>
     <child link="chassis_link" />
     <axis xyz="0 0 1"/>
-    <limit effort="1000" lower="-1000" upper="1000" velocity="2" />
+    <limit effort="1000" lower="-1000" upper="1000" />
   </joint> -->
   <joint name="insert_link_joint" type="fixed">
-    <origin xyz="0 0 0" rpy="0 0 0" />
-    <parent link="panda_link0"/>
-    <child link="insert_link" />
+    <origin xyz="0.05387925 0 0" rpy="0 0 0" />
+    <parent link="insert_link"/>
+    <child link="panda_link0" />
   </joint>
   <link name="insert_link">
@@ -21,5 +21,4 @@
       <origin xyz="0 0 0" rpy="0 0 0" />
       <geometry>
-        <!-- <box size=".2 .2 .2"/> -->
         <mesh filename="$(find mobile_base_description)/meshes/MI_with_TableTop_fixed_origin.stl" scale="0.001 0.001 0.001"/>
       </geometry>
@@ -29,5 +28,5 @@
       <geometry>
         <!-- <box size=".2 .2 .2"/> -->
-        <mesh filename="$(find mobile_base_description)/meshes/MI_with_TableTop_fixed_origin.stl" scale="0.001 0.001 0.001"/>
+        <!-- <mesh filename="$(find mobile_base_description)/meshes/MI_with_TableTop_fixed_origin.stl" scale="0.001 0.001 0.001"/> -->
       </geometry>
     </collision>
@@ -51,12 +50,15 @@
     </joint>
     <link name="arm_${axis_name}_link">
-    <inertial>
-    <origin xyz="0 0 0" rpy="0 0 0" />
-    <mass value="1" />
-    <inertia
-        ixx="1.0" ixy="0.0" ixz="0.0"
-        iyy="1.0" iyz="0.0"
-        izz="1.0" />
-    </inertial>
+      <visual>
+        <origin xyz="0 0 0" rpy="0 0 0" />
+      </visual>
+      <inertial>
+        <origin xyz="0 0 0" rpy="0 0 0" />
+        <mass value="1" />
+      <inertia
+          ixx="1.0" ixy="0.0" ixz="0.0"
+          iyy="1.0" iyz="0.0"
+          izz="1.0" />
+      </inertial>
     </link>
     <transmission name="panda_${axis_name}_transmission">
@@ -70,12 +72,71 @@
     </transmission>
   </xacro:macro>
+ <!--Load revolute joints-->
+  <xacro:macro name="revolute_joint_macro" params="axis_name axis parent child mimic">
+  <joint name="panda_${axis_name}_joint" type="revolute">
+    <!-- <origin xyz="${origin}" rpy="0 0 0" /> -->
+    <limit lower="-1000" upper="1000" effort="1000" velocity="2"/>
+    <parent link="${parent}"/>
+    <child link="${child}" />
+    <axis xyz="${axis}"/>
+    <!-- <limit effort="1000" velocity="2"/> -->
+    <!-- <mimic joint="panda_rx_joint" multiplier="1.0"/> -->
+  </joint>
+    <link name="arm_${axis_name}_link">
+      <inertial>
+        <origin xyz="0 0 0" rpy="0 0 0" />
+        <mass value="1" />
+      <inertia
+        ixx="1.0" ixy="0.0" ixz="0.0"
+        iyy="1.0" iyz="0.0"
+        izz="1.0" />
+      </inertial>
+    </link>
+    <transmission name="panda_${axis_name}_transmission">
+      <type>transmission_interface/SimpleTransmission</type>
+      <joint name="panda_${axis_name}_joint">
+          <hardwareInterface>hardware_interface/VelocityJointInterface</hardwareInterface>
+      </joint>
+      <actuator name="panda_${axis_name}_joint_motor">
+          <mechanicalReduction>1</mechanicalReduction>
+      </actuator>
+    </transmission>
+  </xacro:macro>
   <xacro:prismatic_joint_macro axis_name="x" origin="$(arg origin)" axis="1 0 0" parent="world" child="arm_x_link"/>
   <xacro:prismatic_joint_macro axis_name="y" axis="0 1 0" parent="arm_x_link" child="arm_y_link"/>
-  <xacro:prismatic_joint_macro axis_name="z" axis="0 0 1" parent="arm_y_link" child="arm_z_link"/>
+  <xacro:revolute_joint_macro axis_name="rx" axis="1 0 0" parent="arm_z_link" child="arm_rx_link" mimic='true'/>
+  <xacro:revolute_joint_macro axis_name="ry" axis="0 1 0" parent="arm_rx_link" child="arm_ry_link" mimic="false"/>
+  <joint name="panda_z_joint" type="prismatic">
+    <origin xyz="0 0 0" rpy="0 0 0" />
+    <parent link="arm_y_link"/>
+    <child link="arm_z_link" />
+    <axis xyz="0 0 1"/>
+    <limit effort="1000" lower="-100" upper="100" velocity="2"/>
+  </joint>
+  <link name="arm_z_link">
+    <inertial>
+      <origin xyz="0 0 0" rpy="0 0 0" />
+      <mass value="1" />
+      <inertia
+          ixx="1.0" ixy="0.0" ixz="0.0"
+          iyy="1.0" iyz="0.0"
+          izz="1.0" />
+    </inertial>
+  </link>
+  <transmission name="panda_z_transmission">
+    <type>transmission_interface/SimpleTransmission</type>
+    <joint name="panda_z_joint">
+        <hardwareInterface>hardware_interface/VelocityJointInterface</hardwareInterface>
+    </joint>
+    <actuator name="panda_z_joint_motor">
+        <mechanicalReduction>1</mechanicalReduction>
+    </actuator>
+  </transmission>
+  <!-- <xacro:prismatic_joint_macro axis_name="z" axis="0 0 1" parent="arm_y_link" child="arm_z_link"/> -->
   <!-- Load world rotation joint -->
   <joint name="panda_z_rotation_joint" type="continuous">
     <origin xyz="0 0 0" rpy="0 0 0" />
-    <parent link="arm_z_link"/>
-    <child link="panda_link0" />
+    <parent link="arm_ry_link"/>
+    <child link="insert_link" />
     <axis xyz="0 0 1"/>
     <limit effort="1000.0" velocity="2"/>
@@ -96,4 +157,12 @@
       <robotSimType>gazebo_ros_control/DefaultRobotHWSim</robotSimType>
     </plugin>
+    <!-- <plugin name="gazebo_mimic_joint" filename="libroboticsgroup_upatras_gazebo_mimic_joint_plugin.so">
+      <robotNamespace>/panda</robotNamespace>
+      <gazebo reference="panda_insert"/>
+      <joint>panda_rx_joint</joint>
+      <mimicJoint>panda_ry_joint</mimicJoint>
+      <maxEffort>1000</maxEffort>
+      <hasPID></hasPID>
+    </plugin> -->
   </gazebo>
 </robot>
